File: Schematics/TeslaController/TeslaController.sch (KiCad schematic (older format))
At the start: 93 parts, among them IC1 ATXMEGA256A3-A, P1 PWR_IN, P10 MicroSD, P11 KEYBOARD, P12 INVERTER, P13 DISPLAY, P14 INV_EN, P15 TEMP1, P16 TEMP2, P17 CURRENT_SENS, P2 PWR_OUT1, P3 ESP-12E, P4 ISP, P5 DEBUG, P6 BUZZER, P7 EXPANSION, P8 FAN1, P9 FAN2, Q1 BSS138, Q2 BSS138, Q3 BSS138, Q4 BSS138, Q5 BSS138, Q6 BSS138, Q7 BSS138, Q8 BSS138, Q9 BSS138, U1 AP1117, U2 AP1117D50, U3 AP1117D33, U4 TL431DBZ, Y1 DSX321SH

Commit message: Decided to send the controller PCB off to China rather than etching myself. So fixed up the silkscreen and reduced via sizes a bit.
Parts:
- P1: footprint MyConnectors:ScrewTerm2.54-3 -> MyConnectors:PinHeader_1x03
Changed lines of the file:
@@
 F 0 "P1" H 1050 6550 50  0000 C CNN
 F 1 "PWR_IN" V 1150 6350 50  0000 C CNN
-F 2 "MyConnectors:ScrewTerm2.54-3" H 1050 6350 50  0001 C CNN
+F 2 "MyConnectors:PinHeader_1x03" H 1050 6350 50  0001 C CNN
 F 3 "" H 1050 6350 50  0000 C CNN
 	1    1050 6350

Commit message: - Changed the value of R30 & R31 to up the current sense reference voltage from 0.5V to 1.65V. - TeslaTuner now show current limits in Amps rather than a number between 0 and 4095.
Parts:
- R30: value 1k2 -> 470
- R31: value 300 -> 910
Other:
- note added: "1.65V"
- note removed: "0.5V"
Changed lines of the file:
@@
 P 12600 8450
 F 0 "R30" H 12630 8470 50  0000 L CNN
-F 1 "1k2" H 12630 8410 50  0000 L CNN
+F 1 "470" H 12630 8410 50  0000 L CNN
 F 2 "MyResistors:R_0603" H 12600 8450 50  0001 C CNN
 F 3 "" H 12600 8450 50  0000 C CNN
@@
 P 12600 9250
 F 0 "R31" H 12630 9270 50  0000 L CNN
-F 1 "300" H 12630 9210 50  0000 L CNN
+F 1 "910" H 12630 9210 50  0000 L CNN
 F 2 "MyResistors:R_0603" H 12600 9250 50  0001 C CNN
 F 3 "" H 12600 9250 50  0000 C CNN
@@
 $EndComp
 Text Notes 12650 9000 0    60   ~ 0
-0.5V
+1.65V
 $Comp
 L CP1_Small C12
